File: EEProject.kicad_sch (KiCad schematic)
At the start: 1 part, among them U1 74AHC04

Commit message: dwa
Parts:
- added U2: 74AHC244, symbol 74xx:74AHC244
Changed lines of the file:
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@@
+		)
+	)
+	(symbol
+		(lib_id "74xx:74AHC244")
+		(at 176.53 99.06 0)
+		(unit 1)
+		(exclude_from_sim no)
+		(in_bom yes)
+		(on_board yes)
+		(dnp no)
+		(fields_autoplaced yes)
+		(property "Reference" "U2"
+			(at 178.7241 78.74 0)
+			(effects
+				(font
+					(size 1.27 1.27)
+				)
+				(justify left)
+			)
+		)
+		(property "Value" "74AHC244"
+			(at 178.7241 81.28 0)
+			(effects
+				(font
+					(size 1.27 1.27)
+				)
+				(justify left)
+			)
+		)
+		(property "Footprint" ""
+			(at 176.53 99.06 0)
+			(effects
+				(font
+					(size 1.27 1.27)
+				)
+				(hide yes)
+			)
+		)
+		(property "Datasheet" "https://assets.nexperia.com/documents/data-sheet/74AHC_AHCT244.pdf"
+			(at 176.53 99.06 0)
+			(effects
+				(font
+					(size 1.27 1.27)
+				)
+				(hide yes)
+			)
+		)
+		(property "Description" "8-bit Buffer/Line Driver 3-state"
+			(at 176.53 99.06 0)
+			(effects
+				(font
+					(size 1.27 1.27)
+				)
+				(hide yes)
+			)
+		)
+		(pin "11"
+		)
+		(pin "12"
+		)
+		(pin "13"
+		)
+		(pin "1"
+		)
+		(pin "14"
+		)
+		(pin "10"
+		)
+		(pin "8"
+		)
+		(pin "15"
+		)
+		(pin "6"
+		)
+		(pin "9"
+		)
+		(pin "17"
+		)
+		(pin "2"
+		)
+		(pin "7"
+		)
+		(pin "5"
+		)
+		(pin "20"
+		)
+		(pin "16"
+		)
+		(pin "3"
+		)
+		(pin "19"
+		)
+		(pin "18"
+		)
+		(pin "4"
+		)
+		(instances
+			(project ""
+				(path "/3aa1ef99-b297-42d2-a07b-7cd664ecf53c"
+					(reference "U2")
+					(unit 1)
+				)
+			)
 		)
 	)

Commit message: ds
Parts:
- added U3: 74AHC244, symbol 74xx:74AHC244
Changed lines of the file:
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@@
+		)
+	)
+	(symbol
+		(lib_id "74xx:74AHC244")
+		(at 106.68 138.43 0)
+		(unit 1)
+		(exclude_from_sim no)
+		(in_bom yes)
+		(on_board yes)
+		(dnp no)
+		(fields_autoplaced yes)
+		(property "Reference" "U3"
+			(at 108.8741 118.11 0)
+			(effects
+				(font
+					(size 1.27 1.27)
+				)
+				(justify left)
+			)
+		)
+		(property "Value" "74AHC244"
+			(at 108.8741 120.65 0)
+			(effects
+				(font
+					(size 1.27 1.27)
+				)
+				(justify left)
+			)
+		)
+		(property "Footprint" ""
+			(at 106.68 138.43 0)
+			(effects
+				(font
+					(size 1.27 1.27)
+				)
+				(hide yes)
+			)
+		)
+		(property "Datasheet" "https://assets.nexperia.com/documents/data-sheet/74AHC_AHCT244.pdf"
+			(at 106.68 138.43 0)
+			(effects
+				(font
+					(size 1.27 1.27)
+				)
+				(hide yes)
+			)
+		)
+		(property "Description" "8-bit Buffer/Line Driver 3-state"
+			(at 106.68 138.43 0)
+			(effects
+				(font
+					(size 1.27 1.27)
+				)
+				(hide yes)
+			)
+		)
+		(pin "7"
+		)
+		(pin "5"
+		)
+		(pin "2"
+		)
+		(pin "19"
+		)
+		(pin "11"
+		)
+		(pin "17"
+		)
+		(pin "8"
+		)
+		(pin "13"
+		)
+		(pin "4"
+		)
+		(pin "14"
+		)
+		(pin "6"
+		)
+		(pin "3"
+		)
+		(pin "1"
+		)
+		(pin "16"
+		)
+		(pin "12"
+		)
+		(pin "9"
+		)
+		(pin "10"
+		)
+		(pin "18"
+		)
+		(pin "20"
+		)
+		(pin "15"
+		)
+		(instances
+			(project ""
+				(path "/3aa1ef99-b297-42d2-a07b-7cd664ecf53c"
+					(reference "U3")
+					(unit 1)
+				)
+			)
 		)
 	)
