File: Boost Converter.kicad_sch (KiCad schematic)
At the start: 0 parts

Commit message: 11.10.2024
Parts:
- added C9: 100u, symbol Device:C
- added D2: D_Schottky, symbol Device:D_Schottky
- added L1: L, symbol Device:L
- added Q3: NMOS, symbol Simulation_SPICE:NMOS
Connections:
- new net: D2.2 (A), L1.2, Q3.1 (D)
- new net 30V: C9.1, D2.1 (K)
- new net BCSW: Q3.2 (G)
- new net GND: C9.2, Q3.3 (S)
- new net VCC: L1.1
